File: Chargerv1.brd (EAGLE design)
At the start: 25.4 x 93.7 mm, 12 parts, among them J1 POWER_JACKPTH_LOCK, U1 MCP73831, X1 USB-MICROB

Commit message: Routed Board
Parts:
- added JP2: M023.5MM, SparkFun-Connectors:SCREWTERMINAL-3.5MM-2
- added STANDOFF1, STANDOFF2, STANDOFF3, STANDOFF4: STAND-OFF, SparkFun-Electromechanical:STAND-OFF
- moved D1 49.5 mm to (12.7, 41.9), turned to 270 degrees
- moved C1 39.7 mm to (16.5, 47.0)
- moved C2 37.2 mm to (7.62, 49.5), turned to 180 degrees
- moved R2 37.2 mm to (7.62, 44.5)
- moved R1 37.2 mm to (7.62, 47.0)
- moved U1 37.2 mm to (12.7, 47.0)
- moved X1 20.9 mm to (1.27, 71.1), turned to 270 degrees
- moved JP1 18.7 mm to (22.2, 71.8), turned to 270 degrees
- moved J1 9.92 mm to (12.7, 87.6)
- moved JP3 8.89 mm to (22.9, 78.7)
- flipped B1 to the bottom
Connections:
- net 5V: now also JP2.1
- net GND: now also JP2.2
Routing:
- net V_BATT: track 0.00 -> 86.4 mm
- net 5V: track 0.00 -> 48.9 mm
- net N$1: track 0.00 -> 4.90 mm
- net N$2: track 0.00 -> 4.31 mm
- net N$7: track 0.00 -> 3.32 mm
- added copper zone on layer 16, net 5V
- added copper zone on layer 1, net GND
Other:
- board size 25.4 x 93.7 mm -> 25.4 x 87.3 mm
- board text added: "+"
- board text added: "-"
- board text added: "Single Cell Lipo Charger"
- board text added: "VBATT"
- board text added: "Vin"

Commit message: Ready for Itead order
Final version with gerbers as sent to Itead (ordered 1/30, received
2/11)
Parts:
- removed X1: USB-MICROB, SparkFun-Connectors:USB-MICROB
- added JP4: USB_MICROB_PLUGCONN-11752, SparkFun-Connectors:USB-B-MICRO-SMD_V03
- C1, C2: value (none) -> 4.7uF; device SparkFun-Passives:0603-CAP -> SparkFun-Capacitors:0603-CAP
- R1: value (none) -> 2.0k; device SparkFun-Passives:0603-RES -> SparkFun-Resistors:0603-RES
- R2: value (none) -> 330; device SparkFun-Passives:0603-RES -> SparkFun-Resistors:0603-RES
- moved FRAME1 75.8 mm to (-8.89, -8.89)
Connections:
- net 5V: now also JP4.VBUS1; no longer X1.VBUS
- net GND: now also JP4.GND1; no longer X1.GND, X1.MT1, X1.MT2
Routing:
- net GND: track 0.00 -> 1.12 mm
Changed lines of the file:
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@@
 <?xml version="1.0" encoding="utf-8"?>
 <!DOCTYPE eagle SYSTEM "eagle.dtd">
-<eagle version="6.5.0">
+<eagle version="7.2.0">
 <drawing>
 <settings>
@@
 <layer number="23" name="tOrigins" color="15" fill="1" visible="yes" active="yes"/>
 <layer number="24" name="bOrigins" color="15" fill="1" visible="yes" active="yes"/>
-<layer number="25" name="tNames" color="7" fill="1" visible="yes" active="yes"/>
+<layer number="25" name="tNames" color="7" fill="1" visible="no" active="yes"/>
 <layer number="26" name="bNames" color="7" fill="1" visible="yes" active="yes"/>
 <layer number="27" name="tValues" color="7" fill="1" visible="yes" active="yes"/>
@@
 <layer number="45" name="Holes" color="7" fill="1" visible="no" active="yes"/>
 <layer number="46" name="Milling" color="3" fill="1" visible="no" active="yes"/>
-<layer number="47" name="Measures" color="7" fill="1" visible="no" active="yes"/>
+<layer number="47" name="Measures" color="7" fill="1" visible="yes" active="yes"/>
 <layer number="48" name="Document" color="7" fill="1" visible="yes" active="yes"/>
 <layer number="49" name="Reference" color="7" fill="1" visible="yes" active="yes"/>
@@
 <layer number="56" name="wert" color="7" fill="1" visible="no" active="no"/>
 <layer number="57" name="tCAD" color="7" fill="1" visible="no" active="no"/>
-<layer number="90" name="Modules" color="5" fill="1" visible="yes" active="yes"/>
+<layer number="90" name="Modules" color="5" fill="1" visible="no" active="no"/>
 <layer number="91" name="Nets" color="2" fill="1" visible="no" active="no"/>
 <layer number="92" name="Busses" color="1" fill="1" visible="no" active="no"/>
@@
 <pass name="Default">
 <param name="RoutingGrid" value="50mil"/>
+<param name="AutoGrid" value="1"/>
+<param name="Efforts" value="0"/>
+<param name="TopRouterVariant" value="1"/>
 <param name="tpViaShape" value="round"/>
 <param name="PrefDir.1" value="|"/>
@@
 </autorouter>
 <elements>
-<element name="U1" library="SparkFun-PowerIC" package="SOT23-5" value="MCP73831" x="12.7" y="46.99" rot="R90">
+<element name="U1" library="SparkFun-PowerIC" package="SOT23-5" value="MCP73831" x="12.7" y="46.99" smashed="yes" rot="R90">
 <attribute name="PROD_ID" value="IC-09995" x="78.74" y="99.06" size="1.778" layer="27" rot="R90" display="off"/>
-</element>
-<element name="R1" library="SparkFun-Passives" package="0603-RES" value="" x="7.62" y="46.99"/>
-<element name="R2" library="SparkFun-Passives" package="0603-RES" value="" x="7.62" y="44.45"/>
-<element name="C1" library="SparkFun-Passives" package="0603-CAP" value="" x="16.51" y="46.99" rot="R270"/>
-<element name="C2" library="SparkFun-Passives" package="0603-CAP" value="" x="7.62" y="49.53" rot="R180"/>
-<element name="FRAME1" library="SparkFun-Aesthetics" package="CREATIVE_COMMONS" value="" x="66.04" y="2.54">
-<attribute name="VERSION" value="v01" x="143.51" y="-49.53" size="1.778" layer="27" display="off"/>
-<attribute name="DESIGNER" value="Michelle" x="143.51" y="-49.53" size="1.778" layer="27" display="off"/>
-</element>
-<element name="JP1" library="SparkFun-Connectors" package="JST-2-SMD" value="M02-JST-2MM-SMT" x="22.225" y="71.755" rot="R270">
+<attribute name="NAME" x="10.541" y="46.101" size="0.4064" layer="25" rot="R90"/>
+<attribute name="VALUE" x="13.6525" y="49.0855" size="0.4064" layer="27" rot="R180"/>
+</element>
+<element name="R1" library="SparkFun-Resistors" package="0603-RES" value="2.0k" x="7.62" y="46.99">
+<attribute name="PROD_ID" value="RES-08296" x="7.62" y="46.99" size="1.778" layer="27" display="off"/>
+<attribute name="VALUE" value="2.0k" x="7.62" y="46.99" size="1.778" layer="27" display="off"/>
+</element>
+<element name="R2" library="SparkFun-Resistors" package="0603-RES" value="330" x="7.62" y="44.45">
+<attribute name="PROD_ID" value="RES-00818" x="7.62" y="44.45" size="1.778" layer="27" display="off"/>
+<attribute name="VALUE" value="330" x="7.62" y="44.45" size="1.778" layer="27" display="off"/>
+</element>
+<element name="C1" library="SparkFun-Capacitors" package="0603-CAP" value="4.7uF" x="16.51" y="46.99" rot="R270">
+<attribute name="PROD_ID" value="CAP-08280" x="16.51" y="46.99" size="1.778" layer="27" rot="R270" display="off"/>
+<attribute name="VALUE" value="4.7uF" x="16.51" y="46.99" size="1.778" layer="27" rot="R270" display="off"/>
+</element>
+<element name="C2" library="SparkFun-Capacitors" package="0603-CAP" value="4.7uF" x="7.62" y="49.53" smashed="yes" rot="R180">
+<attribute name="NAME" x="7.239" y="50.673" size="0.4064" layer="25" font="vector" rot="R180"/>
+<attribute name="VALUE" value="4.7uF" x="8.636" y="50.673" size="0.4064" layer="27" font="vector" rot="R180"/>
+<attribute name="PROD_ID" value="CAP-08280" x="7.62" y="49.53" size="1.778" layer="27" rot="R180" display="off"/>
+</element>
+<element name="FRAME1" library="SparkFun-Aesthetics" package="CREATIVE_COMMONS" value="" x="-8.89" y="-8.89" smashed="yes">
+<attribute name="VERSION" value="v01" x="16.51" y="34.29" size="1.27" layer="16" font="vector" ratio="15" rot="SMR270"/>
+<attribute name="DESIGNER" value="Michelle" x="17.78" y="-8.89" size="1.778" layer="51"/>
+</element>
+<element name="JP1" library="SparkFun-Connectors" package="JST-2-SMD" value="M02-JST-2MM-SMT" x="22.225" y="71.755" smashed="yes" rot="R270">
 <attribute name="PROD_ID" value="CONN-08352" x="-48.895" y="53.975" size="1.778" layer="27" rot="R270" display="off"/>
-</element>
-<element name="JP3" library="SparkFun-Connectors" package="SCREWTERMINAL-3.5MM-2" value="M023.5MM" x="22.86" y="78.74" rot="R90"/>
+<attribute name="NAME" x="23.495" y="73.025" size="0.4064" layer="25" rot="R270"/>
+<attribute name="VALUE" x="22.225" y="74.295" size="0.4064" layer="27" rot="R270"/>
+</element>
+<element name="JP3" library="SparkFun-Connectors" package="SCREWTERMINAL-3.5MM-2" value="M023.5MM" x="22.86" y="78.74" smashed="yes" rot="R90">
+<attribute name="NAME" x="20.32" y="77.47" size="0.4064" layer="25" rot="R90"/>
+<attribute name="VALUE" x="20.955" y="79.375" size="0.4064" layer="27" rot="R90"/>
+</element>
 <element name="J1" library="SparkFun-Connectors" package="POWER_JACK_PTH_LOCK" value="POWER_JACKPTH_LOCK" x="12.7" y="87.63" rot="R180">
 <attribute name="SF_ID" value="PRT-00119" x="-6.35" y="121.92" size="1.778" layer="27" rot="R180" display="off"/>
 <attribute name="PROD_ID" value="CONN-08197" x="-6.35" y="121.92" size="1.778" layer="27" rot="R180" display="off"/>
 </element>
-<element name="X1" library="SparkFun-Connectors" package="USB-MICROB" value="USB-MICROB" x="1.27" y="71.12" rot="R270">
-<attribute name="PROD_ID" value="CONN-09505" x="-67.31" y="26.67" size="1.778" layer="27" rot="R270" display="off"/>
-</element>
 <element name="D1" library="SparkFun-LED" package="LED-0603" value="Yellow" x="12.7" y="41.91" rot="R270">
 <attribute name="PROD_ID" value="DIO-09003" x="-53.34" y="-12.7" size="1.778" layer="27" rot="R270" display="off"/>
 </element>
 <element name="B1" library="Battery Holder 18650" package="18650-HOLDER" value="BATTERY18650" x="12.7" y="34.29" rot="MR90"/>
-<element name="JP2" library="SparkFun-Connectors" package="SCREWTERMINAL-3.5MM-2" value="M023.5MM" x="2.54" y="82.55" rot="R270"/>
+<element name="JP2" library="SparkFun-Connectors" package="SCREWTERMINAL-3.5MM-2" value="M023.5MM" x="2.54" y="82.55" smashed="yes" rot="R270">
+<attribute name="NAME" x="5.08" y="83.82" size="0.4064" layer="25" rot="R270"/>
+<attribute name="VALUE" x="4.445" y="81.915" size="0.4064" layer="27" rot="R270"/>
+</element>
 <element name="STANDOFF1" library="SparkFun-Electromechanical" package="STAND-OFF" value="STAND-OFF" x="22.86" y="60.96"/>
 <element name="STANDOFF2" library="SparkFun-Electromechanical" package="STAND-OFF" value="STAND-OFF" x="2.54" y="60.96"/>
 <element name="STANDOFF3" library="SparkFun-Electromechanical" package="STAND-OFF" value="STAND-OFF" x="2.54" y="11.43"/>
 <element name="STANDOFF4" library="SparkFun-Electromechanical" package="STAND-OFF" value="STAND-OFF" x="22.86" y="11.43"/>
+<element name="JP4" library="SparkFun-Connectors" package="USB-B-MICRO-SMD_V03" value="USB_MICROB_PLUGCONN-11752" x="1.27" y="71.12">
+<attribute name="PROD_ID" value="CONN-11752" x="1.27" y="71.12" size="1.778" layer="27" display="off"/>
+</element>
 </elements>
 <signals>
@@
 <signal name="GND">
 <contactref element="C2" pad="2"/>
-<contactref element="X1" pad="GND"/>
-<contactref element="X1" pad="MT1"/>
-<contactref element="X1" pad="MT2"/>
 <contactref element="U1" pad="2"/>
 <contactref element="R1" pad="1"/>
@@
 <vertex x="25.4" y="0"/>
 </polygon>
+<contactref element="JP4" pad="GND1"/>
+<wire x1="3.97" y1="69.82" x2="5.05" y2="69.82" width="0.254" layer="1"/>
+<wire x1="5.05" y1="69.82" x2="5.08" y2="69.85" width="0.254" layer="1"/>
 </signal>
 <signal name="N$7">
@@
 <signal name="5V">
 <contactref element="J1" pad="PWR"/>
-<contactref element="X1" pad="VBUS"/>
 <contactref element="C2" pad="1"/>
 <contactref element="U1" pad="4"/>
@@
 <wire x1="5.08" y1="58.42" x2="6.35" y2="59.69" width="0.254" layer="1"/>
 <wire x1="6.35" y1="59.69" x2="6.35" y2="71.12" width="0.254" layer="1"/>
-<wire x1="3.92" y1="72.42" x2="5.05" y2="72.42" width="0.254" layer="1"/>
 <wire x1="5.05" y1="72.42" x2="6.35" y2="71.12" width="0.254" layer="1"/>
 <wire x1="12.7" y1="73.7522" x2="12.7" y2="73.66" width="0.254" layer="1"/>
 <wire x1="12.7" y1="73.66" x2="10.16" y2="71.12" width="0.254" layer="1"/>
 <wire x1="10.16" y1="71.12" x2="6.35" y2="71.12" width="0.254" layer="1"/>
+<contactref element="JP4" pad="VBUS1"/>
+<wire x1="3.97" y1="72.42" x2="5.05" y2="72.42" width="0.254" layer="1"/>
 </signal>
 <signal name="V_BATT">
